File: Rockets/Schematic.brd (EAGLE design)
At the start: 160 x 100 mm, 9 parts, among them IC1 LM2937

Commit message: WIP
Parts:
- moved BMP1 292.1 mm to (174.0, 2.54)
- moved GPS1 264.5 mm to (186.7, 21.6), turned to 270 degrees
- moved RFM69HCW1 222.5 mm to (142.2, 25.4)
- moved MPU1 202.8 mm to (102.9, 3.81)
- moved MPU2 181.1 mm to (120.7, 3.81)
- moved ESP1 144.5 mm to (99.1, 29.2), turned to 270 degrees
- moved IC1 108.4 mm to (10.2, 17.8), turned to 270 degrees
- moved J1 108.1 mm to (2.54, 2.54), turned to 90 degrees
- moved MICROSD1 103.6 mm to (39.4, 1.27), turned to 90 degrees
Other:
- board size 160 x 100 mm -> 212.1 x 32.7 mm

Commit message: Everthing added needs resistors
Parts:
- removed IC1: LM2937, linear:TO263-3
- added U$1: V_REG_LD1117VXX, SparkFun-IC-Power:TO-220-ALT2
Connections:
- removed net N$19: MICROSD1.CS
- removed net N$20: MICROSD1.DO
- removed net N$21: MICROSD1.CLK
- removed net N$22: MICROSD1.DI
- removed net N$23: MPU1.SCL
- removed net N$26: MPU1.SDA
- removed net N$29: MPU1.ADD
- removed net N$33: MPU2.SCL
- removed net N$34: MPU2.SDA
- removed net N$38: MPU2.ADD
- removed net N$5: BMP1.SCL
- removed net N$6: BMP1.SDA
- removed net N$8: BMP1.SDO
- removed net SCLK: ESP1.ESP32_49, RFM69HCW1.SCK
- new net CLK: ESP1.ESP_12, MICROSD1.CLK, RFM69HCW1.SCK
- new net SCL: BMP1.SCL, ESP1.ESP_17, MPU1.SCL, MPU2.SCL
- new net SDA: BMP1.SDA, ESP1.ESP_14, MPU1.SDA, MPU2.SDA
- new net SDCS: ESP1.ESP32_48, MICROSD1.CS
- net 3.3V: now also BMP1.SDO, U$1.OUT; no longer IC1.3
- net 5V: now also MPU2.ADD, U$1.IN; no longer IC1.1
- net GND: now also MPU1.ADD, U$1.GND; no longer ESP1.ESP_2, IC1.2
- net MISO: now also ESP1.ESP_13, MICROSD1.DO; no longer ESP1.ESP32_50
- net MOSI: now also ESP1.D23, MICROSD1.DI; no longer ESP1.ESP32_51
- net RADIOCS: now also ESP1.ESP32_41
- net RX: now also ESP1.ESP_9; no longer ESP1.ESP_6
- net TX: now also ESP1.ESP_10; no longer ESP1.ESP_7
Routing:
- net 3.3V: track 0.00 -> 220.1 mm, vias 0 -> 2
- net 5V: track 0.00 -> 204.7 mm
- net TX: track 0.00 -> 177.6 mm, vias 0 -> 3
- net SCL: track 0.00 -> 157.8 mm, vias 0 -> 4
- net SDA: track 0.00 -> 152.6 mm, vias 0 -> 3
- net MISO: track 0.00 -> 147.2 mm, vias 0 -> 4
- net RX: track 0.00 -> 133.3 mm
- net MOSI: track 0.00 -> 122.3 mm, vias 0 -> 3
- net CLK: track 0.00 -> 119.1 mm, vias 0 -> 1
- net RADIOCS: track 0.00 -> 110.7 mm
- net SDCS: track 0.00 -> 48.7 mm, vias 0 -> 1
- added copper zone on layer 16, net GND
Other:
- board size 212.1 x 32.7 mm -> 250 x 30 mm

Commit message: Mk1 completed?
Parts:
- removed RFM69HCW1: RFM69HCW, awesome:RFM69HCW
- added C1, C2, C3, C4, C5, C6: 0.1uF, SparkFun-Capacitors:CAP-PTH-SMALL-KIT
- added D1: (no value), SparkFun-LED:LED_3MM-NS
- added R1, R2, R3, R4, R5, R7: (no value), SparkFun-Resistors:AXIAL-0.3
- moved MICROSD1 160.0 mm to (199.4, 2.27)
- moved GPS1 108.7 mm to (79.3, 4.41), turned to 90 degrees
- moved MPU2 103.9 mm to (222.3, 25.2), turned to 180 degrees
- moved MPU1 86.0 mm to (16.9, 4.81)
- moved ESP1 43.0 mm to (142.1, 29.2)
- moved BMP1 25.2 mm to (149.0, 5.54)
- moved U$1 9.43 mm to (8.00, 15.0)
- moved J1 2.83 mm to (4.54, 4.54)
Connections:
- removed net N$18: MICROSD1.CD
- removed net N$9: RFM69HCW1.RST
- new net N$1: ESP1.ESP_12, R3.P$1
- new net N$2: D1.A, ESP1.ESP32_45
- new net SDCD: ESP1.ESP32_42, MICROSD1.CD
- net 3.3V: now also C4.1, C6.1, R1.P$2, R7.P$2
- net 5V: now also C1.1, C2.1, C3.2, C5.2; no longer RFM69HCW1.VIN
- net CLK: now also R3.P$2; no longer ESP1.ESP_12, RFM69HCW1.SCK
- net GND: now also C1.2, C2.2, C3.1, C4.2, C5.1, C6.2, R4.P$1; no longer RFM69HCW1.GND
- net MISO: now also R5.P$2; no longer MICROSD1.DO, RFM69HCW1.MISO
- net MOSI: now also R2.P$1, R2.P$2; no longer RFM69HCW1.MOSI
- net N$3: now also D1.K, R4.P$2; no longer RFM69HCW1.EN
- net N$4: now also MICROSD1.DO, R5.P$1; no longer RFM69HCW1.G0
- net RADIOCS: no longer RFM69HCW1.CS
- net SCL: now also R1.P$1
- net SDA: now also R7.P$1
Routing:
- net GND: track 0.00 -> 283.9 mm
- net TX: track 177.6 -> 42.2 mm, vias 3 -> 0
- net SDCD: track 0.00 -> 128.0 mm, vias 0 -> 3
- net RADIOCS: track 110.7 -> 0.00 mm
- net SDA: track 152.6 -> 258.4 mm, vias 3 -> 1
- net N$2: track 0.00 -> 89.4 mm
- net RX: track 133.3 -> 46.0 mm
- net 5V: track 204.7 -> 290.3 mm, vias 0 -> 1
- net SCL: track 157.8 -> 225.9 mm, vias 4 -> 5
- net CLK: track 119.1 -> 52.2 mm, vias 1 -> 0
- net N$1: track 0.00 -> 63.9 mm, vias 0 -> 1
- net SDCS: track 48.7 -> 84.4 mm, vias 1 -> 2
- net MISO: track 147.2 -> 112.0 mm, vias 4 -> 2
- net N$3: track 0.00 -> 22.1 mm
- net 3.3V: track 220.1 -> 201.9 mm
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Other:
- board size 250 x 30 mm -> 230 x 30 mm
- board text added: "YAR MK1"
- board text added: "created by Asim"

Commit message: Updated the schematics from discord zip
Parts:
- removed U$1: V_REG_LD1117VXX, SparkFun-IC-Power:TO-220-ALT2
- added J2: (no value), SparkFun-Connectors:1X02
- moved J1 10.2 mm to (6.54, 14.5)
- moved MPU1 7.00 mm to (9.87, 4.81)
- moved BMP1 7.00 mm to (142.0, 5.54)
- moved C1 7.00 mm to (8.00, 23.0)
- moved C2 7.00 mm to (139.0, 4.00)
- moved C3 7.00 mm to (195.0, 8.00)
- moved C4 7.00 mm to (74.0, 22.0)
- moved C5 7.00 mm to (218.0, 7.00)
- moved C6 7.00 mm to (156.0, 18.0)
- moved D1 7.00 mm to (27.0, 27.0)
- moved ESP1 7.00 mm to (135.1, 29.2)
- moved GPS1 7.00 mm to (72.3, 4.41)
- moved MICROSD1 7.00 mm to (192.4, 2.27)
- moved MPU2 7.00 mm to (215.3, 25.2)
- moved R1 7.00 mm to (66.0, 28.0)
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Connections:
- new net N$5: ESP1.D23, R2.P$1
- net 3.3V: now also J2.1; no longer U$1.OUT
- net 5V: no longer U$1.IN
- net GND: now also J2.2; no longer U$1.GND
- net MOSI: no longer ESP1.D23, R2.P$1
Routing:
- net GND: track 283.9 -> 21.0 mm, vias 0 -> 2
- net N$5: track 0.00 -> 69.1 mm, vias 0 -> 2
- net MOSI: track 107.5 -> 44.4 mm, vias 2 -> 0
- net 5V: track 290.3 -> 339.6 mm, vias 1 -> 6
- net RX: track 46.0 -> 69.8 mm, vias 0 -> 2
- net SCL: track 225.9 -> 245.1 mm, vias 5 -> 4
- net N$1: track 63.9 -> 45.5 mm, vias 1 -> 2
- net N$2: track 89.4 -> 103.9 mm, vias 0 -> 2
- net SDCD: track 128.0 -> 116.2 mm
- net SDCS: track 84.4 -> 95.5 mm
- net TX: track 42.2 -> 48.2 mm, vias 0 -> 1
- net SDA: track 258.4 -> 262.8 mm, vias 1 -> 6
- net MISO: track 112.0 -> 113.9 mm, vias 2 -> 4
- net 3.3V: track 201.9 -> 200.6 mm, vias 2 -> 6
- net CLK: track 52.2 -> 53.1 mm, vias 0 -> 2
Other:
- board size 230 x 30 mm -> 225 x 30 mm
- board text added: "BMP280"
- board text added: "GPS"
- board text added: "SD Card"
